File: timer-pcb-chargeur/timer-pcb-stepper.kicad_pcb (KiCad board)
At the start: 4 copper layers, 46 x 41 mm, 7 parts, among them J11 JST_04, J3 On/off

Commit message: mise à jour fichier kicad stepper + led. création dossier chargeur PCB.création du fichier .rpt
Connections:
- J11 pad 1: +5V -> GND
- U1 pad 1: +5V -> GND
Routing:
- net GND: track 0.00 -> 16.9 mm
- net +5V: track 35.3 -> 18.4 mm
Changed lines of the file:
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@@
 	(net 3 "5V_chargeur_input")
 	(net 4 "On{slash}off")
+	(net 5 "GND")
 	(footprint "1_My_Custom_Library:TP4056_chargeur_USB-C"
 		(layer "F.Cu")
@@
 			(layers "F.Cu" "F.Mask" "F.Paste")
 			(roundrect_rratio 0.15)
-			(net 1 "+5V")
+			(net 5 "GND")
 			(pinfunction "out-")
 			(pintype "power_out")
@@
 			(remove_unused_layers no)
 			(roundrect_rratio 0.208333)
-			(net 1 "+5V")
+			(net 5 "GND")
 			(pintype "passive")
 		)
@@
 	)
 	(segment
-		(start 142.45 70.85)
-		(end 143.275 70.025)
-		(width 0.7)
-		(layer "F.Cu")
-		(net 1)
-	)
-	(segment
-		(start 139.65 70.85)
-		(end 142.45 70.85)
-		(width 0.7)
-		(layer "F.Cu")
-		(net 1)
-	)
-	(segment
 		(start 149.8 84.35)
 		(end 156.05 84.35)
-		(width 0.7)
-		(layer "F.Cu")
-		(net 1)
-	)
-	(segment
-		(start 143.275 70.025)
-		(end 156.225 70.025)
 		(width 0.7)
 		(layer "F.Cu")
@@
 		(net 4)
 	)
+	(segment
+		(start 142.45 70.85)
+		(end 143.275 70.025)
+		(width 0.7)
+		(layer "F.Cu")
+		(net 5)
+	)
+	(segment
+		(start 139.65 70.85)
+		(end 142.45 70.85)
+		(width 0.7)
+		(layer "F.Cu")
+		(net 5)
+	)
+	(segment
+		(start 143.275 70.025)
+		(end 156.225 70.025)
+		(width 0.7)
+		(layer "F.Cu")
+		(net 5)
+	)
 	(zone
